Commit message: Modificacion del urdf para el nuevo jnt_antebrazo_palma

File: src/xolobot_arm/models/xolobot.urdf (robot description, URDF)
Before this commit: robot xolobot_arm, 7 links, 6 joints
Joints:
- added joint jnt_antebrazo_palma: type revolute, parent link_antebrazo_izq, child link_palma_izq, origin xyz=0 0 0.100 rpy=0 0 0, axis 0 0 1, limit lower=-3.1416 upper=3.1416 effort=1000 velocity=1000

Commit message: Correccion de texturas del antebrazo, palma, base, soporte

File: src/xolobot_arm/models/xolobot.urdf (robot description, URDF)
Before this commit: robot xolobot_arm, 7 links, 7 joints
Links:
- added link link_palma_izq
Joints:
- joint jnt_palma_pulgar_1: parent link_antebrazo_izq -> link_palma_izq

Commit message: Se mueve y simula que agarra la lata

File: src/xolobot_arm/models/xolobot.urdf (robot description, URDF)
Before this commit: robot xolobot_arm, 8 links, 7 joints
Links:
- added link link_indice_1_izq
Joints:
- added joint jnt_palma_indice_1: type revolute, parent link_palma_izq, child link_indice_1_izq, origin xyz=0.0119  0.00435  0 rpy=0 0 0, axis 0 0 -1, limit lower=0.0 upper=1.45 effort=8000 velocity=2

Commit message: Version final

File: src/xolobot_arm/models/xolobot.urdf (robot description, URDF)
Before this commit: robot xolobot_arm, 9 links, 8 joints
Links:
- added link link_anular_1_izq
- added link link_cordial_1_izq
- added link link_menique_1_izq
- added link link_pulgar_2_izq
- added link link_pulgar_3_izq
Joints:
- added joint jnt_palma_cordial_1: type revolute, parent link_palma_izq, child link_cordial_1_izq, origin xyz=0.0119  0.00435  0 rpy=0 0 0, axis 0 0 -1, limit lower=0.0 upper=1.45 effort=8000 velocity=2
- added joint jnt_palma_jnt_palma_anular_1indice_1: type revolute, parent link_palma_izq, child link_anular_1_izq, origin xyz=0.0119  0.00435  0 rpy=0 0 0, axis 0 0 -1, limit lower=0.0 upper=1.45 effort=8000 velocity=2
- added joint jnt_palma_menique_1: type revolute, parent link_palma_izq, child link_menique_1_izq, origin xyz=0.0119  0.00435  0 rpy=0 0 0, axis 0 0 -1, limit lower=0.0 upper=1.45 effort=8000 velocity=2
- added joint jnt_pulgar_1_2: type revolute, parent link_pulgar_1_izq, child link_pulgar_2_izq, origin xyz=0.0119  0.00435  0 rpy=0 0 0, axis 0 0 -1, limit lower=0.0 upper=1.45 effort=8000 velocity=2
- added joint jnt_pulgar_2_3: type revolute, parent link_pulgar_2_izq, child link_pulgar_3_izq, origin xyz=0.0119  0.00435  0 rpy=0 0 0, axis 0 0 -1, limit lower=0.0 upper=1.45 effort=8000 velocity=2

Commit message: 2 bumpers y 5 dedos

File: src/xolobot_arm/models/xolobot.urdf (robot description, URDF)
Before this commit: robot xolobot_arm, 14 links, 13 joints
Joints:
- removed joint jnt_palma_jnt_palma_anular_1indice_1
- added joint jnt_anular_1_2: type revolute, parent link_anular_1_izq, child link_anular_2_izq, origin xyz=0.0119  0.00435  0 rpy=0 0 0, axis 0 0 -1, limit lower=0.0 upper=1.45 effort=8000 velocity=2
- added joint jnt_anular_2_3: type revolute, parent link_anular_2_izq, child link_anular_3_izq, origin xyz=0.0119  0.00435  0 rpy=0 0 0, axis 0 0 -1, limit lower=0.0 upper=1.45 effort=8000 velocity=2
- added joint jnt_cordial_1_2: type revolute, parent link_cordial_1_izq, child link_cordial_2_izq, origin xyz=0.0119  0.00435  0 rpy=0 0 0, axis 0 0 -1, limit lower=0.0 upper=1.45 effort=8000 velocity=2
- added joint jnt_cordial_2_3: type revolute, parent link_cordial_2_izq, child link_cordial_3_izq, origin xyz=0.0119  0.00435  0 rpy=0 0 0, axis 0 0 -1, limit lower=0.0 upper=1.45 effort=8000 velocity=2
- added joint jnt_indice_1_2: type revolute, parent link_indice_1_izq, child link_indice_2_izq, origin xyz=0.0119  0.00435  0 rpy=0 0 0, axis 0 0 -1, limit lower=0.0 upper=1.45 effort=8000 velocity=2
- added joint jnt_indice_2_3: type revolute, parent link_indice_2_izq, child link_indice_3_izq, origin xyz=0.0119  0.00435  0 rpy=0 0 0, axis 0 0 -1, limit lower=0.0 upper=1.45 effort=8000 velocity=2
- added joint jnt_menique_1_2: type revolute, parent link_menique_1_izq, child link_menique_2_izq, origin xyz=0.0119  0.00435  0 rpy=0 0 0, axis 0 0 -1, limit lower=0.0 upper=1.45 effort=8000 velocity=2
- added joint jnt_menique_2_3: type revolute, parent link_menique_2_izq, child link_menique_3_izq, origin xyz=0.0119  0.00435  0 rpy=0 0 0, axis 0 0 -1, limit lower=0.0 upper=1.45 effort=8000 velocity=2
- added joint jnt_palma_anular_1: type revolute, parent link_palma_izq, child link_anular_1_izq, origin xyz=0.0119  0.00435  0 rpy=0 0 0, axis 0 0 -1, limit lower=0.0 upper=1.45 effort=8000 velocity=2
